File: PID Control Position.kicad_sch (KiCad schematic)
At the start: 29 parts, among them Q1 TIP41C, U1 LM324, U2 LM741

Commit message: added pdf files
Other:
- company: (none) -> KEL. 7
- title: (none) -> PID POSITION CONTROL
- moved on the sheet: C1, C2, C3, Kd1, Ki1, Kp1, Q1, U1B, U1C, U1D, U2, swD1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
